Commit message: updated inertia tensor and add two lines to Move_it_config pacakge

File: custom_kortex_description/grippers/custom_gripper/urdf/custom_gripper_macro.xacro (robot description, xacro)
@@ -27,7 +27,8 @@
                 <mass value="0.5" />
                 <origin xyz="0.0 0.0 0.0" />
-                <inertia ixx = "1.0" ixy = "0.000000" ixz = "0.000000"
-                         iyx = "0.000000" iyy = "1.0" iyz = "0.000000"
-                         izx = "0.000000" izy = "0.000000" izz = "1.0" />
+                <!-- using formula m(3r^2+h^2)/12 -->
+                <inertia ixx = "0.00115" ixy = "0.000000" ixz = "0.000000"
+                         iyx = "0.000000" iyy = "0.00115" iyz = "0.000000"
+                         izx = "0.000000" izy = "0.000000" izz = "0.00115" />
             </inertial>
         </link>
