Commit message: Version 3

File: custom_kortex_description/robots/gen3_custom_gripper.xacro (robot description, xacro)
@@ -2,8 +2,11 @@
 <robot name="gen3_custom_gripper" xmlns:xacro="http://ros.org/wiki/xacro">
     <!-- Arguments -->
-    <xacro:arg name="arm" default="gen3" />
+  	<xacro:arg name="arm" default="gen3" />
+    <xacro:arg name="dof" default="7" />
+    <xacro:arg name="vision" default="true" />
     <xacro:arg name="gripper" default="custom_gripper" />
     <xacro:arg name="sim" default="false" />
+    <xacro:arg name="prefix" default="" />
     <xacro:include filename="$(find custom_kortex_description)/robots/kortex_robot.xacro" />
-    <xacro:load_robot arm="$(arg arm)" gripper="$(arg gripper)" sim="$(arg sim)"/>
+    <xacro:load_robot arm="$(arg arm)" gripper="$(arg gripper)" dof="$(arg dof)" vision="$(arg vision)" sim="$(arg sim)" prefix="$(arg prefix)" />
 </robot>

File: custom_kortex_description/robots/kortex_robot.xacro (robot description, xacro)
@@ -1,11 +1,7 @@
 <?xml version="1.0"?>
 <robot xmlns:xacro="http://ros.org/wiki/xacro">
-    <xacro:macro name="load_robot" params="arm gripper sim">
-        <!-- Arguments -->
-        <xacro:property name="arm" value="$(arg arm)" />
-        <xacro:property name="gripper" default="$(arg gripper)" />
-        <xacro:property name="sim" default="$(arg sim)" />
+    <xacro:macro name="load_robot" params="arm gripper dof vision sim prefix">
         <!-- Files to include -->
-        <xacro:include filename="$(find kortex_description)/arms/$(arg arm)/urdf/$(arg arm)_macro.xacro" />
+        <xacro:include filename="$(find kortex_description)/arms/$(arg arm)/${dof}dof/urdf/$(arg arm)_macro.xacro" />
         <xacro:unless value="${not gripper}">
             <xacro:include filename="$(find custom_kortex_description)/grippers/$(arg gripper)/urdf/$(arg gripper)_macro.xacro" />
@@ -13,5 +9,5 @@
         <xacro:if value="$(arg sim)">
             <!-- Arm transmission elements-->
-            <xacro:include filename="$(find kortex_description)/arms/$(arg arm)/urdf/$(arg arm)_transmission_macro.xacro" />
+            <xacro:include filename="$(find kortex_description)/arms/${arm}/${dof}dof/urdf/${arm}_transmission_macro.xacro" />
             <!-- Gripper transmission elements if there is a gripper-->
             <xacro:unless value="${not gripper}">
@@ -30,5 +26,5 @@
         </xacro:if>
         <!-- Load the arm -->
-        <xacro:load_arm parent="">
+        <xacro:load_arm parent="" dof="${dof}" vision="${vision}" prefix="${prefix}">
             <origin xyz="0 0 0" rpy="0 0 0"/>
         </xacro:load_arm>
@@ -39,5 +35,5 @@
         <!-- Load the Gazebo transmissions and gazebo_ros_control plugin -->
         <xacro:if value="$(arg sim)">
-            <xacro:load_gazebo_arm_transmissions/>
+            <xacro:load_gazebo_arm_transmissions prefix="${prefix}"/>
             <xacro:unless value="${not gripper}">
                 <xacro:load_gazebo_gripper_transmissions/>

File: custom_kortex_description/robots/mobile_kortex_robot.xacro (robot description, xacro)
@@ -1,10 +1,54 @@
 <?xml version="1.0"?>
-<robot name="mobile_kortex_robot" xmlns:xacro="http://ros.org/wiki/xacro">
-    <!-- Arguments -->
-    <xacro:arg name="arm" default="gen3" />
-    <xacro:arg name="gripper" default="custom_gripper" />
-    <xacro:arg name="sim" default="false" />
-    <xacro:include filename="$(find custom_kortex_description)/robots/kortex_robot.xacro" />
-    <xacro:include filename="$(find jackal_description)/urdf/jackal.urdf.xacro" />
-    <xacro:load_robot arm="$(arg arm)" gripper="$(arg gripper)" sim="$(arg sim)"/>
+<robot xmlns:xacro="http://ros.org/wiki/xacro">
+    <xacro:macro name="load_robot" params="arm gripper sim">
+        <!-- Arguments -->
+        <xacro:property name="arm" value="$(arg arm)" />
+        <xacro:property name="gripper" default="$(arg gripper)" />
+        <xacro:property name="sim" default="$(arg sim)" />
+        <xacro:property name="dof" default="7" />
+        <xacro:property name="vision" default="true" />
+        <xacro:property name="prefix" default="" />
+        <!-- Files to include -->
+        <xacro:include filename="$(find kortex_description)/arms/$(arg arm)/7dof/urdf/$(arg arm)_macro.xacro" />
+        <xacro:unless value="${not gripper}">
+            <xacro:include filename="$(find custom_kortex_description)/grippers/$(arg gripper)/urdf/$(arg gripper)_macro.xacro" />
+        </xacro:unless>
+        <xacro:if value="$(arg sim)">
+            <!-- Arm transmission elements-->
+            <xacro:include filename="$(find kortex_description)/arms/$(arg arm)/7dof/urdf/$(arg arm)_transmission_macro.xacro" />
+            <!-- Gripper transmission elements if there is a gripper-->
+            <xacro:unless value="${not gripper}">
+                <xacro:include filename="$(find custom_kortex_description)/grippers/$(arg gripper)/urdf/$(arg gripper)_transmission_macro.xacro" />
+            </xacro:unless>
+        </xacro:if>
+        <!-- Run the macros -->
+        <!-- Load the arm -->
+        <xacro:load_arm parent="${arm_mount}" dof="${dof}" vision="${vision}" prefix="${prefix}">
+            <origin xyz="0 0 0" rpy="0 0 0"/>
+        </xacro:load_arm>
+        <xacro:macro name="jackal_arm_jt">
+            <joint name="jackal_arm_joint" type="fixed">
+                <parent link="${arm_mount}"/>
+                <child link="base_link"/>
+                <origin rpy="0 0 0" xyz="0.0 0.0 0"/>
+            </joint>
+        </xacro:macro>
+        <xacro:jackal_arm_jt/>
+        <!-- Load the gripper -->
+        <xacro:unless value="${not gripper}">
+            <xacro:load_gripper parent="${last_arm_link}"/> <!-- last_arm_link is defined in "$(find kortex_description)/arms/$(arg arm)/urdf/$(arg arm)_macro.xacro" -->
+        </xacro:unless>
+        <!-- Load the Gazebo transmissions and gazebo_ros_control plugin -->
+        <xacro:if value="$(arg sim)">
+            <xacro:load_gazebo_arm_transmissions prefix="${prefix}"/>
+            <xacro:unless value="${not gripper}">
+                <xacro:load_gazebo_gripper_transmissions/>
+            </xacro:unless>
+            <gazebo>
+                <plugin name="gazebo_ros_control" filename="libgazebo_ros_control.so">
+                    <legacyModeNS>true</legacyModeNS>
+                </plugin>
+            </gazebo>
+        </xacro:if>
+    </xacro:macro>
 </robot>
